Commit message: update urdf to attach virtual finger to link 8

File: models/franka_description/robots/frankaEmikaPandaVirtual.urdf (robot description, URDF)
Before this commit: robot panda, 13 links, 12 joints
Joints:
- joint panda_finger_virtual_joint: limit lower=-3.1416 upper=3.1416 effort=0 velocity=1.0 -> lower=-3.1416 upper=3.1416 effort=0 velocity=2.610; origin xyz=0 0 0.1034 rpy=-1.57079632679 0 0 -> xyz=0 0 0.1034 rpy=-1.57079632679 0 -0.785398163397; parent panda_hand -> panda_link8
